File: Projects/Arduino_Fio/Arduino_Fio.kicad_pcb (KiCad board)
At the start: 2 copper layers, 27.9 x 64.8 mm, 2 parts, among them P1 Digital, P2 Analog

Commit message: Update existing templates to version 6
Other:
- net class Default removed
