File: Projects/Arduino_Mega_R3/Arduino_Mega.kicad_pcb (KiCad board)
At the start: 2 copper layers, 101.6 x 53.3 mm, 13 parts, among them P1 Digital, P10 CONN_01X01, P11 CONN_01X01, P12 CONN_01X01, P13 CONN_01X01, P2 Power, P3 Analog, P4 Analog, P5 PWM, P6 PWM, P7 Communication, P8 CONN_01X01, P9 CONN_01X01

Commit message: Update existing templates to version 6
Other:
- net class Default removed
