File: Projects/Arduino_Micro/Arduino_Micro.kicad_pcb (KiCad board)
At the start: 2 copper layers, 17.8 x 48.3 mm, 6 parts, among them P1 Digital, P2 Analog, P3 CONN_01X01, P4 CONN_01X01, P5 CONN_01X01, P6 CONN_01X01

Commit message: Update existing templates to version 6
Other:
- net class Default removed
