File: Projects/Arduino_Mini/Arduino_Mini.kicad_pcb (KiCad board)
At the start: 2 copper layers, 17.8 x 30.5 mm, 6 parts, among them P1 ADC, P2 Digital, P3 ADC, P4 COM, P5 Analog, P6 PWR

Commit message: Update existing templates to version 6
Other:
- net class Default removed
