File: Projects/Arduino_Pro_Mini/Arduino_Pro_Mini.kicad_pcb (KiCad board)
At the start: 2 copper layers, 17.8 x 33 mm, 5 parts, among them P1 Digital, P2 COM, P3 ADC, P4 Analog, P5 ADC

Commit message: Update existing templates to version 6
Other:
- net class Default removed
