File: Projects/Arduino_Pro_Mini/Arduino_Pro_Mini.kicad_pcb (KiCad board)
At the start: 2 copper layers, 33 x 17.8 mm, 5 parts, among them J1 FTDI, J2 I2C, J3 Analog, J6 Digital, J7 Analog

Commit message: Update projects for KiCad version 7
Parts:
- J6: value Digital -> Analog
- J7: value Analog -> Digital
