File: Projects/Arduino_Uno_R3/Arduino_Uno.kicad_pcb (KiCad board)
At the start: 2 copper layers, 68.6 x 53.3 mm, 8 parts, among them P1 Power, P2 Analog, P3 Digital, P4 Digital, P5 CONN_01X01, P6 CONN_01X01, P7 CONN_01X01, P8 CONN_01X01

Commit message: Update existing templates to version 6
Other:
- net class Default removed
