File: Projects/BeagleBone-Black-Cape/BeagleBone-Black-Cape.kicad_pcb (KiCad board)
At the start: 2 copper layers, 54.6 x 86.4 mm, 2 parts, among them P8 BeagleBone_Black_Header, P9 BeagleBone_Black_Header

Commit message: Update existing templates to version 6
Other:
- net class Default removed
