File: Projects/BeagleBone-Black-Cape/BeagleBone-Black-Cape.kicad_pcb (KiCad board)
At the start: 2 copper layers, 86.4 x 54.6 mm, 6 parts, among them P8 BeagleBone_Black_Header, P9 BeagleBone_Black_Header

Commit message: Update projects for KiCad version 7
Connections:
- net /GPIO[117] renamed /GPIO117
- net /GPIO[122] renamed /GPIO122
- net /GPIO[125] renamed /GPIO125
- net /GPIO[14] renamed /GPIO14
- net /GPIO[15] renamed /GPIO15
- net /GPIO[20] renamed /GPIO20
- net /GPIO[22] renamed /GPIO22
- net /GPIO[23] renamed /GPIO23
- net /GPIO[26] renamed /GPIO26
- net /GPIO[27] renamed /GPIO27
- net /GPIO[2] renamed /GPIO2
- net /GPIO[30] renamed /GPIO30
- net /GPIO[31] renamed /GPIO31
- net /GPIO[3] renamed /GPIO3
- net /GPIO[40] renamed /GPIO40
- net /GPIO[44] renamed /GPIO44
- net /GPIO[45] renamed /GPIO45
- net /GPIO[46] renamed /GPIO46
- net /GPIO[47] renamed /GPIO47
- net /GPIO[48] renamed /GPIO48
- net /GPIO[49] renamed /GPIO49
- net /GPIO[4] renamed /GPIO4
- net /GPIO[51] renamed /GPIO51
- net /GPIO[5] renamed /GPIO5
- net /GPIO[60] renamed /GPIO60
- net /GPIO[61] renamed /GPIO61
- net /GPIO[65] renamed /GPIO65
- net /GPIO[66] renamed /GPIO66
- net /GPIO[67] renamed /GPIO67
- net /GPIO[68] renamed /GPIO68
- net /GPIO[69] renamed /GPIO69
- net /GPIO[7] renamed /GPIO7
- net /LCD.DATA[0] renamed /LCD.DATA0
- net /LCD.DATA[10] renamed /LCD.DATA10
- net /LCD.DATA[11] renamed /LCD.DATA11
- net /LCD.DATA[13] renamed /LCD.DATA13
- net /LCD.DATA[14] renamed /LCD.DATA14
- net /LCD.DATA[15] renamed /LCD.DATA15
- net /LCD.DATA[1] renamed /LCD.DATA1
- net /LCD.DATA[2] renamed /LCD.DATA2
- net /LCD.DATA[3] renamed /LCD.DATA3
- net /LCD.DATA[4] renamed /LCD.DATA4
- net /LCD.DATA[5] renamed /LCD.DATA5
- net /LCD.DATA[6] renamed /LCD.DATA6
- net /LCD.DATA[7] renamed /LCD.DATA7
- net /LCD.DATA[8] renamed /LCD.DATA8
- net /LCD.DATA[9] renamed /LCD.DATA9
- net /MMC1.DAT[0] renamed /MMC1.DAT0
- net /MMC1.DAT[1] renamed /MMC1.DAT1
- net /MMC1.DAT[2] renamed /MMC1.DAT2
- net /MMC1.DAT[3] renamed /MMC1.DAT3
- net /MMC1.DAT[4] renamed /MMC1.DAT4
- net /MMC1.DAT[5] renamed /MMC1.DAT5
- net /MMC1.DAT[6] renamed /MMC1.DAT6
- net /MMC1.DAT[7] renamed /MMC1.DAT7
