File: Projects/BeagleBone-Black-Cape/BeagleBone-Black-Cape.kicad_pcb (KiCad board)
At the start: 2 copper layers, 86.4 x 54.6 mm, 6 parts, among them P8 BeagleBone_Black_Header, P9 BeagleBone_Black_Header

Commit message: Correct BeagleBone Black pinout
Connections:
- P8 pad 26: /LCD.PCLK -> /GPIO61
- P8 pad 28: /GPIO61 -> /LCD.PCLK
- P8 pad 35: /LCD.DATA8 -> /LCD.DATA12
- P8 pad 37: /LCD.DATA6 -> /LCD.DATA8
- P8 pad 39: /LCD.DATA4 -> /LCD.DATA6
- P8 pad 41: /LCD.DATA2 -> /LCD.DATA4
- P8 pad 43: /LCD.DATA0 -> /LCD.DATA2
- P8 pad 45: GNDD -> /LCD.DATA0
Changed lines of the file:
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@@
 	(net 80 "/SPI1.SCLK")
 	(net 81 "/SPI1.CS0")
+	(net 82 "/LCD.DATA12")
 	(footprint "Connector_PinHeader_2.54mm:PinHeader_2x23_P2.54mm_Vertical"
 		(locked yes)
@@
 			(layers "*.Cu" "*.Mask")
 			(remove_unused_layers no)
-			(net 21 "/LCD.PCLK")
+			(net 29 "/GPIO61")
 			(pinfunction "Pin_26")
 			(pintype "passive")
@@
 			(layers "*.Cu" "*.Mask")
 			(remove_unused_layers no)
-			(net 29 "/GPIO61")
+			(net 21 "/LCD.PCLK")
 			(pinfunction "Pin_28")
 			(pintype "passive")
@@
 			(layers "*.Cu" "*.Mask")
 			(remove_unused_layers no)
-			(net 34 "/LCD.DATA8")
+			(net 82 "/LCD.DATA12")
 			(pinfunction "Pin_35")
 			(pintype "passive")
@@
 			(layers "*.Cu" "*.Mask")
 			(remove_unused_layers no)
-			(net 36 "/LCD.DATA6")
+			(net 34 "/LCD.DATA8")
 			(pinfunction "Pin_37")
 			(pintype "passive")
@@
 			(layers "*.Cu" "*.Mask")
 			(remove_unused_layers no)
-			(net 38 "/LCD.DATA4")
+			(net 36 "/LCD.DATA6")
 			(pinfunction "Pin_39")
 			(pintype "passive")
@@
 			(layers "*.Cu" "*.Mask")
 			(remove_unused_layers no)
-			(net 40 "/LCD.DATA2")
+			(net 38 "/LCD.DATA4")
 			(pinfunction "Pin_41")
 			(pintype "passive")
@@
 			(layers "*.Cu" "*.Mask")
 			(remove_unused_layers no)
-			(net 42 "/LCD.DATA0")
+			(net 40 "/LCD.DATA2")
 			(pinfunction "Pin_43")
 			(pintype "passive")
@@
 			(layers "*.Cu" "*.Mask")
 			(remove_unused_layers no)
-			(net 50 "GNDD")
+			(net 42 "/LCD.DATA0")
 			(pinfunction "Pin_45")
 			(pintype "passive")
