File: Projects/EuroCard160mmX100mm/EuroCard160mmX100mm.kicad_pcb (KiCad board)
At the start: 2 copper layers, 160 x 100 mm, 4 parts

Commit message: Update projects for KiCad version 7
Changed lines of the file:
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@@
-(kicad_pcb (version 20211014) (generator pcbnew)
+(kicad_pcb (version 20221018) (generator pcbnew)
   (general
     (thickness 1.6)
@@
       (layer "F.SilkS" (type "Top Silk Screen"))
       (layer "F.Paste" (type "Top Solder Paste"))
-      (layer "F.Mask" (type "Top Solder Mask") (color "Green") (thickness 0.01))
+      (layer "F.Mask" (type "Top Solder Mask") (color "Green") (color "Green") (thickness 0.01))
       (layer "F.Cu" (type "copper") (thickness 0.035))
       (layer "dielectric 1" (type "core") (thickness 1.51) (material "FR4") (epsilon_r 4.5) (loss_tangent 0.02))
       (layer "B.Cu" (type "copper") (thickness 0.035))
-      (layer "B.Mask" (type "Bottom Solder Mask") (color "Green") (thickness 0.01))
+      (layer "B.Mask" (type "Bottom Solder Mask") (color "Green") (color "Green") (thickness 0.01))
       (layer "B.Paste" (type "Bottom Solder Paste"))
       (layer "B.SilkS" (type "Bottom Silk Screen"))
@@
     (pcbplotparams
       (layerselection 0x0000030_ffffffff)
+      (plot_on_all_layers_selection 0x0000000_00000000)
       (disableapertmacros false)
       (usegerberextensions false)
@@
       (usegerberadvancedattributes true)
       (creategerberjobfile true)
-      (svguseinch false)
+      (dashed_line_dash_ratio 12.000000)
+      (dashed_line_gap_ratio 3.000000)
       (svgprecision 6)
-      (excludeedgelayer true)
       (plotframeref false)
       (viasonmask false)
@@
     (attr exclude_from_pos_files exclude_from_bom)
     (fp_text reference "MH4" (at 0 -3.35) (layer "F.SilkS") hide
-      (effects (font (size 1 1) (thickness 0.15)))
+        (effects (font (size 1 1) (thickness 0.15)))
     )
     (fp_text value "MountingHole_2.7mm_M2.5_DIN965" (at 0 3.35) (layer "F.Fab") hide
-      (effects (font (size 1 1) (thickness 0.15)))
+        (effects (font (size 1 1) (thickness 0.15)))
     )
     (fp_text user "${REFERENCE}" (at 0.3 0) (layer "F.Fab") hide
-      (effects (font (size 1 1) (thickness 0.15)))
+        (effects (font (size 1 1) (thickness 0.15)))
     )
-    (fp_circle (center 0 0) (end 2.35 0) (layer "Cmts.User") (width 0.15) (fill none))
-    (fp_circle (center 0 0) (end 2.6 0) (layer "F.CrtYd") (width 0.05) (fill none))
-    (pad "" np_thru_hole circle locked (at 0 0) (size 2.7 2.7) (drill 2.7) (layers *.Cu *.Mask))
+    (fp_circle (center 0 0) (end 2.35 0)
+      (stroke (width 0.15) (type solid)) (fill none) (layer "Cmts.User"))
+    (fp_circle (center 0 0) (end 2.6 0)
+      (stroke (width 0.05) (type solid)) (fill none) (layer "F.CrtYd"))
+    (pad "" np_thru_hole circle locked (at 0 0) (size 2.7 2.7) (drill 2.7) (layers "*.Cu" "*.Mask"))
   )
   (footprint "MountingHole:MountingHole_2.7mm_M2.5_DIN965" (layer "F.Cu")
@@
     (attr exclude_from_pos_files exclude_from_bom)
     (fp_text reference "MH1" (at 0 -3.35) (layer "F.SilkS") hide
-      (effects (font (size 1 1) (thickness 0.15)))
+        (effects (font (size 1 1) (thickness 0.15)))
     )
     (fp_text value "MountingHole_2.7mm_M2.5_DIN965" (at 0 3.35) (layer "F.Fab") hide
-      (effects (font (size 1 1) (thickness 0.15)))
+        (effects (font (size 1 1) (thickness 0.15)))
     )
     (fp_text user "${REFERENCE}" (at 0.3 0) (layer "F.Fab") hide
-      (effects (font (size 1 1) (thickness 0.15)))
+        (effects (font (size 1 1) (thickness 0.15)))
     )
-    (fp_circle (center 0 0) (end 2.35 0) (layer "Cmts.User") (width 0.15) (fill none))
-    (fp_circle (center 0 0) (end 2.6 0) (layer "F.CrtYd") (width 0.05) (fill none))
-    (pad "" np_thru_hole circle locked (at 0 0) (size 2.7 2.7) (drill 2.7) (layers *.Cu *.Mask))
+    (fp_circle (center 0 0) (end 2.35 0)
+      (stroke (width 0.15) (type solid)) (fill none) (layer "Cmts.User"))
+    (fp_circle (center 0 0) (end 2.6 0)
+      (stroke (width 0.05) (type solid)) (fill none) (layer "F.CrtYd"))
+    (pad "" np_thru_hole circle (at 0 0) (size 2.7 2.7) (drill 2.7) (layers "*.Cu" "*.Mask"))
   )
   (footprint "MountingHole:MountingHole_2.7mm_M2.5_DIN965" locked (layer "F.Cu")
@@
     (attr exclude_from_pos_files exclude_from_bom)
     (fp_text reference "MH2" (at 0 -3.35) (layer "F.SilkS") hide
-      (effects (font (size 1 1) (thickness 0.15)))
+        (effects (font (size 1 1) (thickness 0.15)))
     )
     (fp_text value "MountingHole_2.7mm_M2.5_DIN965" (at 0 3.35) (layer "F.Fab") hide
-      (effects (font (size 1 1) (thickness 0.15)))
+        (effects (font (size 1 1) (thickness 0.15)))
     )
     (fp_text user "${REFERENCE}" (at 0.3 0) (layer "F.Fab") hide
-      (effects (font (size 1 1) (thickness 0.15)))
+        (effects (font (size 1 1) (thickness 0.15)))
     )
-    (fp_circle (center 0 0) (end 2.35 0) (layer "Cmts.User") (width 0.15) (fill none))
-    (fp_circle (center 0 0) (end 2.6 0) (layer "F.CrtYd") (width 0.05) (fill none))
-    (pad "" np_thru_hole circle locked (at 0 0) (size 2.7 2.7) (drill 2.7) (layers *.Cu *.Mask))
+    (fp_circle (center 0 0) (end 2.35 0)
+      (stroke (width 0.15) (type solid)) (fill none) (layer "Cmts.User"))
+    (fp_circle (center 0 0) (end 2.6 0)
+      (stroke (width 0.05) (type solid)) (fill none) (layer "F.CrtYd"))
+    (pad "" np_thru_hole circle locked (at 0 0) (size 2.7 2.7) (drill 2.7) (layers "*.Cu" "*.Mask"))
   )
   (footprint "MountingHole:MountingHole_2.7mm_M2.5_DIN965" locked (layer "F.Cu")
@@
     (attr exclude_from_pos_files exclude_from_bom)
     (fp_text reference "MH3" (at 0 -3.35) (layer "F.SilkS") hide
-      (effects (font (size 1 1) (thickness 0.15)))
+        (effects (font (size 1 1) (thickness 0.15)))
     )
     (fp_text value "MountingHole_2.7mm_M2.5_DIN965" (at 0 3.35) (layer "F.Fab") hide
-      (effects (font (size 1 1) (thickness 0.15)))
+        (effects (font (size 1 1) (thickness 0.15)))
     )
     (fp_text user "${REFERENCE}" (at 0.3 0) (layer "F.Fab") hide
-      (effects (font (size 1 1) (thickness 0.15)))
+        (effects (font (size 1 1) (thickness 0.15)))
     )
-    (fp_circle (center 0 0) (end 2.35 0) (layer "Cmts.User") (width 0.15) (fill none))
-    (fp_circle (center 0 0) (end 2.6 0) (layer "F.CrtYd") (width 0.05) (fill none))
-    (pad "" np_thru_hole circle locked (at 0 0) (size 2.7 2.7) (drill 2.7) (layers *.Cu *.Mask))
+    (fp_circle (center 0 0) (end 2.35 0)
+      (stroke (width 0.15) (type solid)) (fill none) (layer "Cmts.User"))
+    (fp_circle (center 0 0) (end 2.6 0)
+      (stroke (width 0.05) (type solid)) (fill none) (layer "F.CrtYd"))
+    (pad "" np_thru_hole circle locked (at 0 0) (size 2.7 2.7) (drill 2.7) (layers "*.Cu" "*.Mask"))
   )
-  (gr_rect locked (start 55 145) (end 215 45) (layer "Edge.Cuts") (width 0.15) (fill none))
+  (gr_rect locked (start 55 45) (end 215 145)
+    (stroke (width 0.15) (type solid)) (fill none) (layer "Edge.Cuts"))
   (gr_text "Mounting holes are optional\nKeepout areas are for for guide rails" (at 55.5 148) (layer "Cmts.User")
     (effects (font (size 1 1) (thickness 0.15)) (justify left))
   )
-  (zone (net 0) (net_name "") (layers F&B.Cu) (hatch full 0.508)
+  (zone (net 0) (net_name "") (layers "F&B.Cu") (hatch full 0.508)
     (connect_pads (clearance 0))
-    (min_thickness 0.254)
-    (keepout (tracks not_allowed) (vias not_allowed) (pads not_allowed ) (copperpour allowed) (footprints not_allowed))
+    (min_thickness 0.254) (filled_areas_thickness no)
+    (keepout (tracks not_allowed) (vias not_allowed) (pads not_allowed) (copperpour allowed) (footprints not_allowed))
     (fill (thermal_gap 0.508) (thermal_bridge_width 0.508))
     (polygon
@@
     )
   )
-  (zone (net 0) (net_name "") (layers F&B.Cu) (hatch full 0.508)
+  (zone (net 0) (net_name "") (layers "F&B.Cu") (hatch full 0.508)
     (connect_pads (clearance 0))
-    (min_thickness 0.254)
-    (keepout (tracks not_allowed) (vias not_allowed) (pads not_allowed ) (copperpour allowed) (footprints not_allowed))
+    (min_thickness 0.254) (filled_areas_thickness no)
+    (keepout (tracks not_allowed) (vias not_allowed) (pads not_allowed) (copperpour allowed) (footprints not_allowed))
     (fill (thermal_gap 0.508) (thermal_bridge_width 0.508))
     (polygon
