File: Projects/EuroCard160mmX100mm_holes/EuroCard160mmX100mm_holes.kicad_pcb (KiCad board)
At the start: 2 copper layers, 159.9 x 99.9 mm, 4 parts

Commit message: Update existing templates to version 6
Other:
- net class Default removed
