File: Projects/Hammond_1593K_Enclosure/Hammond_1593K_Enclosure.kicad_pcb (KiCad board)
At the start: 2 copper layers, 56.6 x 57.7 mm, 4 parts

Commit message: Update existing templates to version 6
Other:
- net class Default removed
