File: Projects/raspberrypi-gpio/raspberrypi-gpio.kicad_pcb (KiCad board)
At the start: 2 copper layers, 85 x 56 mm, 1 part, among them P1 CONN_13X2

Commit message: Update existing templates to version 6
Other:
- net class Default removed
- net class Power removed
