File: Projects/raspberrypi-gpio-40pin/raspberrypi-gpio-40pin.kicad_pcb (KiCad board)
At the start: 2 copper layers, 65 x 56 mm, 5 parts, among them P1 Conn_02x20_Odd_Even

Commit message: Update existing templates to version 6
Other:
- net class Default removed
- net class Power removed
