File: Projects/stm32f100-discovery-shield/stm32f100-discovery-shield.kicad_pcb (KiCad board)
At the start: 2 copper layers, 43.2 x 84.5 mm, 3 parts, among them P1 CONN28, P2 CONN28, P3 CONN6

Commit message: Update existing templates to version 6
Other:
- net class Default removed
