File: Projects/ti-stellaris-boosterpack40_min/boosterpack40_min.kicad_pcb (KiCad board)
At the start: 2 copper layers, 50.8 x 34.3 mm, 4 parts, among them J1 TI_BOOSTER_40_J1, J2 TI_BOOSTER_40_J2, J3 TI_BOOSTER_40_J3, J4 TI_BOOSTER_40_J4

Commit message: Update existing templates to version 6
Other:
- net class Default removed
