File: Projects/TI-LaunchPad-BoosterPack-20pin/TI-LaunchPad-BoosterPack-20pin.kicad_pcb (KiCad board)
At the start: 2 copper layers, 50.8 x 34.3 mm, 3 parts, among them J1 Conn_01x10, J2 Conn_01x10

Commit message: Update projects for KiCad version 7
Connections:
- net /*D[19] renamed /*D19
- net /D[10]/SDA renamed /D10/SDA
- net /D[11] renamed /D11
- net /D[12]/SPI.CS renamed /D12/SPI.CS
- net /D[13]/SPI.CS renamed /D13/SPI.CS
- net /D[14]/SPI.MISO renamed /D14/SPI.MISO
- net /D[15]/SPI.MOSI renamed /D15/SPI.MOSI
- net /D[17] renamed /D17
- net /D[18]/SPI.CS renamed /D18/SPI.CS
- net /D[2]/A renamed /D2/A
- net /D[3]/UART.RX renamed /D3/UART.RX
- net /D[4]/UART.TX renamed /D4/UART.TX
- net /D[5] renamed /D5
- net /D[6]/A renamed /D6/A
- net /D[7]/SPI.CLK renamed /D7/SPI.CLK
- net /D[8] renamed /D8
- net /D[9]/SCL renamed /D9/SCL
- net /RST/D[16] renamed /RST/D16
